File: bridge1.kicad_sch (KiCad schematic)
At the start: 0 parts

Commit message: Initial schematic design for bridge
Parts:
- added J1: Conn_01x04, Connector_PinHeader_2.54mm:PinHeader_1x04_P2.54mm_Vertical, symbol Connector_Generic:Conn_01x04
- added R1: 150, Resistor_SMD:R_1206_3216Metric_Pad1.30x1.75mm_HandSolder, symbol Device:R
- added U1: pico, Wayne:RaspberryPi_Pico_Common_Unspecified, symbol Wayne:pico
Connections:
- new net: R1.1, U1.21 (GP16)
- new net: J1.3 (Pin_3), U1.22 (GP17)
- new net: J1.1 (Pin_1), U1.39 (VSYS)
- new net: J1.4 (Pin_4), R1.2
- new net GND: J1.2 (Pin_2), U1.13 (GND), U1.18 (GND), U1.23 (GND), U1.28 (GND), U1.3 (GND), U1.33 (GND), U1.38 (GND), U1.8 (GND)
- no-connect marks 0 -> 29
Other:
- title: (none) -> Bridge1 - a UART to WiFi bridge using Pico2W.

Commit message: Updated schematic and project files with full design
Parts:
- added C1: 220uF, symbol Device:C_Polarized
- added C2: 100uF, symbol Device:C_Polarized
- added C3, C4: 1.0uF, Capacitor_SMD:C_1206_3216Metric, symbol Device:C
- added C5: 0.1uF, Capacitor_SMD:C_1206_3216Metric, symbol Device:C
- added D1: SS14, Diode_SMD:D_SMA, symbol Device:D_Schottky
- added FB1: BLM41, Inductor_SMD:L_1206_3216Metric_Pad1.22x1.90mm_HandSolder, symbol Device:FerriteBead
Connections:
- net GND: now also C1.2, C2.2, C3.2, C4.2, C5.2
- net uart_rx: now reaches J1.3 (Pin_3), U1.22 (GP17)
- net at U1.39 (VSYS): now also C2.1, C4.1, C5.1, D1.1 (K); no longer J1.1 (Pin_1)
- net uart_tx: now reaches J1.4 (Pin_4), R1.2
- new net: C1.1, C3.1, D1.2 (A), FB1.1
- new net: FB1.2, J1.1 (Pin_1)
Other:
- moved on the sheet: J1, R1, U1
